File: pcb/NivelesDeNivelesSensor.kicad_pcb (KiCad board)
At the start: 2 copper layers, 6 parts, among them J1 JAE_SIM_Card_SF72S006, U1 SIM800C, U2 LP3947, U3 ATmega32L-8P, U5 FT232RL

Commit message: pcb updates
Routing:
- net GND: track 0.00 -> 138.9 mm
- net +5V: track 0.00 -> 89.0 mm, vias 0 -> 1
- net unconnected-(J1-PadSH): track 0.00 -> 44.8 mm
- net Net-(U3-PA0): track 0.00 -> 43.1 mm
- net Net-(U3-PA1): track 0.00 -> 37.7 mm
- net Net-(U1-UART1_RXD): track 0.00 -> 23.6 mm
- net Net-(U1-UART1_TXD): track 0.00 -> 21.3 mm
- net /C1: track 0.00 -> 12.1 mm
- net /C6: track 0.00 -> 11.4 mm
- net /C3: track 0.00 -> 8.88 mm
- net /C2: track 0.00 -> 6.18 mm
Other:
- board outline added: 43.2 x 58.4 mm
