File: pcb/NivelesDeNivelesSensor.kicad_pcb (KiCad board)
At the start: 2 copper layers, 43.2 x 58.4 mm, 6 parts, among them J1 JAE_SIM_Card_SF72S006, U1 SIM800C, U2 LP3947, U3 ATmega32L-8P, U5 FT232RL

Commit message: small updates
Connections:
- U3 pad 22: unconnected-(U3-PC0-Pad22) -> Net-(U3-PC0)
- U3 pad 23: unconnected-(U3-PC1-Pad23) -> Net-(U3-PC1)
- U3 pad 24: unconnected-(U3-PC2-Pad24) -> Net-(MK1--)
- U3 pad 25: unconnected-(U3-PC3-Pad25) -> Net-(MK1-+)
Changed lines of the file:
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@@
 	(net 65 "unconnected-(U3-PD6-Pad20)")
 	(net 66 "unconnected-(U3-PD7-Pad21)")
-	(net 67 "unconnected-(U3-PC0-Pad22)")
-	(net 68 "unconnected-(U3-PC1-Pad23)")
-	(net 69 "unconnected-(U3-PC2-Pad24)")
-	(net 70 "unconnected-(U3-PC3-Pad25)")
+	(net 67 "Net-(MK1--)")
+	(net 68 "Net-(MK1-+)")
+	(net 69 "Net-(U3-PC0)")
+	(net 70 "Net-(U3-PC1)")
 	(net 71 "unconnected-(U3-PC4-Pad26)")
 	(net 72 "unconnected-(U3-PC5-Pad27)")
@@
 			)
 		)
-		(property "Datasheet" ""
+		(property "Datasheet" "https://www.jae.com/direct/topics/topics_file_download/topics_id=68892&ext_no=06&index=0&_lang=en&v=202003111511468456809"
 			(at 0 0 0)
 			(unlocked yes)
@@
 			)
 		)
-		(property "Description" "Nano-SIM Card (4FF) connector with Detect Switch"
+		(property "Description" ""
 			(at 0 0 0)
 			(unlocked yes)
@@
 			)
 		)
+		(property ki_fp_filters "JAE*SIM*Card*SF72S006*")
+		(sheetname "Root")
 		(sheetfile "NivelesDeNivelesSensor.kicad_sch")
 		(attr smd)
@@
 			)
 		)
-		(property "Datasheet" ""
+		(property "Datasheet" "http://simcom.ee/documents/SIM800C/SIM800C_Hardware_Design_V1.05.pdf"
 			(at 0 0 0)
 			(unlocked yes)
@@
 			)
 		)
-		(property "Description" "GSM Quad-Band Communication Module, GPRS, Audio Engine, AT Command Set, Bluetooth is Optional"
+		(property "Description" ""
 			(at 0 0 0)
 			(unlocked yes)
@@
 			)
 		)
+		(property ki_fp_filters "SIMCom*SIM800C*")
+		(sheetname "Root")
 		(sheetfile "NivelesDeNivelesSensor.kicad_sch")
 		(attr smd)
@@
 			)
 		)
-		(property "Datasheet" ""
+		(property "Datasheet" "http://www.onsemi.com/pub_link/Collateral/MBR0520LT1-D.PDF"
 			(at 0 0 0)
 			(unlocked yes)
@@
 			)
 		)
-		(property "Description" "20V 0.5A Schottky Power Rectifier Diode, SOD-123"
+		(property "Description" ""
 			(at 0 0 0)
 			(unlocked yes)
@@
 			)
 		)
+		(property ki_fp_filters "D*SOD?123*")
+		(sheetname "Root")
 		(sheetfile "NivelesDeNivelesSensor.kicad_sch")
 		(attr smd)
@@
 			)
 		)
-		(property "Datasheet" ""
+		(property "Datasheet" "http://ww1.microchip.com/downloads/en/DeviceDoc/doc2503.pdf"
 			(at 0 0 0)
 			(unlocked yes)
@@
 			)
 		)
-		(property "Description" "8MHz, 32kB Flash, 2kB SRAM, 1kB EEPROM, JTAG, DIP-40"
+		(property "Description" ""
 			(at 0 0 0)
 			(unlocked yes)
@@
 			)
 		)
+		(property ki_fp_filters "DIP*W15.24mm*")
+		(sheetname "Root")
 		(sheetfile "NivelesDeNivelesSensor.kicad_sch")
 		(attr through_hole)
@@
 			(layers "*.Cu" "*.Mask")
 			(remove_unused_layers no)
-			(net 67 "unconnected-(U3-PC0-Pad22)")
+			(net 69 "Net-(U3-PC0)")
 			(pinfunction "PC0")
 			(pintype "bidirectional")
@@
 			(layers "*.Cu" "*.Mask")
 			(remove_unused_layers no)
-			(net 68 "unconnected-(U3-PC1-Pad23)")
+			(net 70 "Net-(U3-PC1)")
 			(pinfunction "PC1")
 			(pintype "bidirectional")
@@
 			(layers "*.Cu" "*.Mask")
 			(remove_unused_layers no)
-			(net 69 "unconnected-(U3-PC2-Pad24)")
+			(net 67 "Net-(MK1--)")
 			(pinfunction "PC2")
 			(pintype "bidirectional")
@@
 			(layers "*.Cu" "*.Mask")
 			(remove_unused_layers no)
-			(net 70 "unconnected-(U3-PC3-Pad25)")
+			(net 68 "Net-(MK1-+)")
 			(pinfunction "PC3")
 			(pintype "bidirectional")
@@
 			)
 		)
-		(property "Datasheet" ""
+		(property "Datasheet" "https://www.ftdichip.com/Support/Documents/DataSheets/ICs/DS_FT232R.pdf"
 			(at 0 0 0)
 			(unlocked yes)
@@
 			)
 		)
-		(property "Description" "USB to Serial Interface, SSOP-28"
+		(property "Description" ""
 			(at 0 0 0)
 			(unlocked yes)
@@
 			)
 		)
+		(property ki_fp_filters "SSOP*5.3x10.2mm*P0.65mm*")
+		(sheetname "Root")
 		(sheetfile "NivelesDeNivelesSensor.kicad_sch")
 		(attr smd)
@@
 			)
 		)
-		(property "Datasheet" ""
+		(property "Datasheet" "http://www.ti.com/lit/ds/symlink/lp3947.pdf"
 			(at 0 0 0)
 			(unlocked yes)
@@
 			)
 		)
-		(property "Description" "Single Cell Li-Ion LDO Battery Charger IC, Up to 1A, Support USB charging scheme"
+		(property "Description" ""
 			(at 0 0 0)
 			(unlocked yes)
@@
 			)
 		)
+		(property ki_fp_filters "WSON*4.0x4.0mm*P0.5mm*")
+		(sheetname "Root")
 		(sheetfile "NivelesDeNivelesSensor.kicad_sch")
 		(attr smd)
