File: pcb/NivelesDeNivelesSensor.kicad_sch (KiCad schematic)
At the start: 21 parts, among them J1 JAE_SIM_Card_SF72S006, J2 USB_C_Receptacle, SW1 SW_Push, U1 SIM800C, U2 LP3947, U3 ATmega32L-8P, U5 FT232RL

Commit message: stuff
Parts:
- added SC1: Solar_Cell, symbol Device:Solar_Cell
Connections:
- net +5V: now also SC1.1 (+)
- net GND: now also SC1.2 (-)
Changed lines of the file:
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@@
+    )
+  )
+  (symbol (lib_id "power:+5V") (at 194.31 128.27 0) (unit 1)
+    (in_bom yes) (on_board yes) (dnp no) (fields_autoplaced)
+    (property "Reference" "#PWR016" (at 194.31 132.08 0)
+      (effects (font (size 1.27 1.27)) hide)
+    )
+    (property "Value" "+5V" (at 194.31 123.19 0)
+      (effects (font (size 1.27 1.27)))
+    )
+    (property "Footprint" "" (at 194.31 128.27 0)
+      (effects (font (size 1.27 1.27)) hide)
+    )
+    (property "Datasheet" "" (at 194.31 128.27 0)
+      (effects (font (size 1.27 1.27)) hide)
+    )
+    (pin "1")
+    (instances
+      (project "NivelesDeNivelesSensor"
+        (path "/e47ae6ce-fa48-474b-854f-61bc182e962e"
+          (reference "#PWR016") (unit 1)
+        )
+      )
     )
   )
@@
     )
   )
+  (symbol (lib_id "power:GND") (at 194.31 135.89 0) (unit 1)
+    (in_bom yes) (on_board yes) (dnp no) (fields_autoplaced)
+    (property "Reference" "#PWR015" (at 194.31 142.24 0)
+      (effects (font (size 1.27 1.27)) hide)
+    )
+    (property "Value" "GND" (at 194.31 140.97 0)
+      (effects (font (size 1.27 1.27)))
+    )
+    (property "Footprint" "" (at 194.31 135.89 0)
+      (effects (font (size 1.27 1.27)) hide)
+    )
+    (property "Datasheet" "" (at 194.31 135.89 0)
+      (effects (font (size 1.27 1.27)) hide)
+    )
+    (pin "1")
+    (instances
+      (project "NivelesDeNivelesSensor"
+        (path "/e47ae6ce-fa48-474b-854f-61bc182e962e"
+          (reference "#PWR015") (unit 1)
+        )
+      )
+    )
+  )
   (symbol (lib_id "MCU_Microchip_ATmega:ATmega32L-8P") (at 78.74 82.55 0) (unit 1)
     (in_bom yes) (on_board yes) (dnp no) (fields_autoplaced)
@@
         )
       )
+    )
+  )
+  (symbol (lib_id "Device:Solar_Cell") (at 194.31 133.35 0) (unit 1)
+    (in_bom yes) (on_board yes) (dnp no) (fields_autoplaced)
+    (property "Reference" "SC1" (at 198.12 129.921 0)
+      (effects (font (size 1.27 1.27)) (justify left))
+    )
+    (property "Value" "Solar_Cell" (at 198.12 132.461 0)
+      (effects (font (size 1.27 1.27)) (justify left))
+    )
+    (property "Footprint" "" (at 194.31 131.826 90)
+      (effects (font (size 1.27 1.27)) hide)
+    )
+    (property "Datasheet" "~" (at 194.31 131.826 90)
+      (effects (font (size 1.27 1.27)) hide)
+    )
+    (pin "1")
+    (pin "2")
+    (instances
+      (project "NivelesDeNivelesSensor"
+        (path "/e47ae6ce-fa48-474b-854f-61bc182e962e"
+          (reference "SC1") (unit 1)
+        )
+      )
